File: PCIe-USB-hub/PCIe-USB-hub.kicad_pcb (KiCad board)
At the start: 4 copper layers, 0 parts

Commit message: Чут чут модифицировал
Parts:
- added C1: EEEFK1E151P, Capacitor_SMD:C_Elec_8x10.2, F.Cu at (25.3, 38.1)
- added C10: EEEFK1E151P, Capacitor_SMD:C_Elec_8x10.2, F.Cu at (38.6, 77.5)
- added C11: 100nF, Capacitor_SMD:C_0402_1005Metric, F.Cu at (31.4, 104.5)
- added C12: 100nF, Capacitor_SMD:C_0402_1005Metric, F.Cu at (31.4, 106.4)
- added C13: 100nF, Capacitor_SMD:C_0402_1005Metric, F.Cu at (31.4, 108.4)
- added C14: 100nF, Capacitor_SMD:C_0402_1005Metric, F.Cu at (31.4, 110.4)
- added C15: 100nF, Capacitor_SMD:C_0402_1005Metric, F.Cu at (31.4, 112.3)
- added C16: 100nF, Capacitor_SMD:C_0402_1005Metric, F.Cu at (31.4, 114.3)
- added C17: 100nF, Capacitor_SMD:C_0402_1005Metric, F.Cu at (31.4, 116.3)
- added C18: 100nF, Capacitor_SMD:C_0402_1005Metric, F.Cu at (31.4, 118.2)
- added C19: 100nF, Capacitor_SMD:C_0402_1005Metric, F.Cu at (31.4, 120.2)
- added C2: EEEFK1E151P, Capacitor_SMD:C_Elec_8x10.2, F.Cu at (25.3, 48.0)
- added C20: 100nF, Capacitor_SMD:C_0402_1005Metric, F.Cu at (34.3, 104.5)
- added C21: 100nF, Capacitor_SMD:C_0402_1005Metric, F.Cu at (34.3, 106.4)
- added C22: 100nF, Capacitor_SMD:C_0402_1005Metric, F.Cu at (34.3, 108.4)
- added C23: 100nF, Capacitor_SMD:C_0402_1005Metric, F.Cu at (34.3, 110.4)
- added C24: 100nF, Capacitor_SMD:C_0402_1005Metric, F.Cu at (34.3, 112.3)
- added C25: 100nF, Capacitor_SMD:C_0402_1005Metric, F.Cu at (34.3, 114.3)
- added C26: 100nF, Capacitor_SMD:C_0402_1005Metric, F.Cu at (34.3, 116.3)
- added C27: 100nF, Capacitor_SMD:C_0402_1005Metric, F.Cu at (34.3, 118.2)
- added C28: 100nF, Capacitor_SMD:C_0402_1005Metric, F.Cu at (34.3, 120.2)
- added C29: 100nF, Capacitor_SMD:C_0402_1005Metric, F.Cu at (37.2, 104.5)
- added C3: EEEFK1E151P, Capacitor_SMD:C_Elec_8x10.2, F.Cu at (25.3, 57.8)
- added C30: 100nF, Capacitor_SMD:C_0402_1005Metric, F.Cu at (37.2, 106.4)
- added C31: 100nF, Capacitor_SMD:C_0402_1005Metric, F.Cu at (37.2, 108.4)
- added C32: 100nF, Capacitor_SMD:C_0402_1005Metric, F.Cu at (37.2, 110.4)
- added C33: 100nF, Capacitor_SMD:C_0402_1005Metric, F.Cu at (37.2, 112.3)
- added C34: 100nF, Capacitor_SMD:C_0402_1005Metric, F.Cu at (37.2, 114.3)
- added C35: 100nF, Capacitor_SMD:C_0402_1005Metric, F.Cu at (37.2, 116.3)
- added C36: 100nF, Capacitor_SMD:C_0402_1005Metric, F.Cu at (37.2, 118.2)
- added C37: 100nF, Capacitor_SMD:C_0402_1005Metric, F.Cu at (37.2, 120.2)
- added C38: 100nF, Capacitor_SMD:C_0402_1005Metric, F.Cu at (40.1, 104.5)
- added C39: 100nF, Capacitor_SMD:C_0402_1005Metric, F.Cu at (46.6, 50.9)
- added C4: EEEFK1E151P, Capacitor_SMD:C_Elec_8x10.2, F.Cu at (25.3, 67.7)
- added C40: 100nF, Capacitor_SMD:C_0402_1005Metric, F.Cu at (46.6, 52.9)
- added C41: 100nF, Capacitor_SMD:C_0402_1005Metric, F.Cu at (46.6, 54.9)
- added C42: 100nF, Capacitor_SMD:C_0402_1005Metric, F.Cu at (46.6, 56.8)
- added C43: 100nF, Capacitor_SMD:C_0402_1005Metric, F.Cu at (40.1, 106.4)
- added C44: 100nF, Capacitor_SMD:C_0402_1005Metric, F.Cu at (40.1, 108.4)
- added C45: 10pF, Capacitor_SMD:C_0402_1005Metric, F.Cu at (40.1, 110.4)
- added C46: 10pF, Capacitor_SMD:C_0402_1005Metric, F.Cu at (40.1, 112.3)
- added C47: 100nF, Capacitor_SMD:C_0402_1005Metric, F.Cu at (40.1, 114.3)
- added C48: 100nF, Capacitor_SMD:C_0402_1005Metric, F.Cu at (40.1, 116.3)
- added C49: 10pF, Capacitor_SMD:C_0402_1005Metric, F.Cu at (40.1, 118.2)
- added C5: EEEFK1E151P, Capacitor_SMD:C_Elec_8x10.2, F.Cu at (25.3, 77.5)
- added C50: 10pF, Capacitor_SMD:C_0402_1005Metric, F.Cu at (40.1, 120.2)
- added C51: 10pF, Capacitor_SMD:C_0402_1005Metric, F.Cu at (42.9, 104.5)
- added C52: 10pF, Capacitor_SMD:C_0402_1005Metric, F.Cu at (42.9, 106.4)
- added C53: 100nF, Capacitor_SMD:C_0402_1005Metric, F.Cu at (42.9, 108.4)
- added C54: 100nF, Capacitor_SMD:C_0402_1005Metric, F.Cu at (42.9, 110.4)
- added C55: 22uF, Capacitor_SMD:C_0402_1005Metric, F.Cu at (46.6, 58.8)
- added C56: 22uF, Capacitor_SMD:C_0402_1005Metric, F.Cu at (46.6, 60.8)
- added C57: 100nF, Capacitor_SMD:C_0402_1005Metric, F.Cu at (46.6, 62.7)
- added C58: 22uF, Capacitor_SMD:C_0402_1005Metric, F.Cu at (46.6, 64.7)
- added C6: EEEFK1E151P, Capacitor_SMD:C_Elec_8x10.2, F.Cu at (38.6, 38.1)
- added C7: EEEFK1E151P, Capacitor_SMD:C_Elec_8x10.2, F.Cu at (38.6, 48.0)
- added C8: EEEFK1E151P, Capacitor_SMD:C_Elec_8x10.2, F.Cu at (38.6, 57.8)
- added C9: EEEFK1E151P, Capacitor_SMD:C_Elec_8x10.2, F.Cu at (38.6, 67.7)
- added D1: BAT54CW, Package_TO_SOT_SMD:SOT-323_SC-70, F.Cu at (51.8, 105.5)
- added D2: BAT54CW, Package_TO_SOT_SMD:SOT-323_SC-70, F.Cu at (51.8, 109.4)
- added D3: BAT54CW, Package_TO_SOT_SMD:SOT-323_SC-70, F.Cu at (51.8, 113.2)
- added DD2: UPD720210K8-BAF-A, Package_DFN_QFN:QFN-76-1EP_9x9mm_P0.4mm_EP5.81x6.31mm, F.Cu at (24.4, 90.1)
- added DD3: TPS2552DRVR, Package_SON:WSON-6-1EP_2x2mm_P0.65mm_EP1x1.6mm, F.Cu at (53.2, 67.5)
- added DD4: UPD720210K8-BAF-A, Package_DFN_QFN:QFN-76-1EP_9x9mm_P0.4mm_EP5.81x6.31mm, F.Cu at (24.4, 101.4)
- added DD5: MX25L8006EM2I-12G, Package_SO:SOP-8_3.9x4.9mm_P1.27mm, F.Cu at (22.9, 110.4)
- added DD6: MX25L8006EM2I-12G, Package_SO:SOP-8_3.9x4.9mm_P1.27mm, F.Cu at (22.9, 117.0)
- added DD8: MX25L8006EM2I-12G, Package_SO:SOP-8_3.9x4.9mm_P1.27mm, F.Cu at (22.9, 123.6)
- added J2: USB3_A_Stacked, Connector_USB:USB3_A_Molex_48406-0001_Horizontal_Stacked, F.Cu at (24.6, 20.7)
- added J3: USB3_A_Stacked, Connector_USB:USB3_A_Molex_48406-0001_Horizontal_Stacked, F.Cu at (43.2, 20.7)
- added J4: USB3_A_Stacked, Connector_USB:USB3_A_Molex_48406-0001_Horizontal_Stacked, F.Cu at (79.7, 46.5)
- added J5: USB3_A_Stacked, Connector_USB:USB3_A_Molex_48406-0001_Horizontal_Stacked, F.Cu at (80.1, 64.2)
- added J6: USB3_A_Stacked, Connector_USB:USB3_A_Molex_48406-0001_Horizontal_Stacked, F.Cu at (80.0, 82.8)
- added J7: Barrel_Jack_MountingPin, Connector_BarrelJack:BarrelJack_GCT_DCJ200-10-A_Horizontal, F.Cu at (50.7, 35.2)
- added L2: 0.68uH, Inductor_SMD:L_Cenker_CKCS4020, F.Cu at (48.2, 68.5)
- added L3: 3.3uH, PCM_4ms_Inductor:COIL_5040, F.Cu at (55.3, 78.6)
- added R1: 10K, PCM_Resistor_SMD_AKL:R_0603_1608Metric, F.Cu at (32.1, 85.8)
- added R10: 10K, PCM_Resistor_SMD_AKL:R_0603_1608Metric, F.Cu at (36.2, 91.2)
- added R11: 10K, PCM_Resistor_SMD_AKL:R_0603_1608Metric, F.Cu at (36.2, 94.0)
- added R12: 4.7K, PCM_Resistor_SMD_AKL:R_0603_1608Metric, F.Cu at (36.2, 96.7)
- added R13: 4.7K, PCM_Resistor_SMD_AKL:R_0603_1608Metric, F.Cu at (36.2, 99.4)
- added R14: 680, PCM_Resistor_SMD_AKL:R_0603_1608Metric, F.Cu at (36.2, 102.1)
- added R15: 1.6K, PCM_Resistor_SMD_AKL:R_0603_1608Metric, F.Cu at (40.3, 85.8)
- added R16: 1.6K, PCM_Resistor_SMD_AKL:R_0603_1608Metric, F.Cu at (40.3, 88.5)
- added R17: 680, PCM_Resistor_SMD_AKL:R_0603_1608Metric, F.Cu at (40.3, 91.2)
- added R18: 10K, PCM_Resistor_SMD_AKL:R_0603_1608Metric, F.Cu at (40.3, 94.0)
- added R19: 10K, PCM_Resistor_SMD_AKL:R_0603_1608Metric, F.Cu at (40.3, 96.7)
- added R2: 47K, PCM_Resistor_SMD_AKL:R_0603_1608Metric, F.Cu at (32.1, 88.5)
- added R20: 10K, PCM_Resistor_SMD_AKL:R_0603_1608Metric, F.Cu at (40.3, 99.4)
- added R21: 10K, PCM_Resistor_SMD_AKL:R_0603_1608Metric, F.Cu at (40.3, 102.1)
- added R22: 10K, PCM_Resistor_SMD_AKL:R_0603_1608Metric, F.Cu at (44.4, 85.8)
- added R23: 10K, PCM_Resistor_SMD_AKL:R_0603_1608Metric, F.Cu at (44.4, 88.5)
- added R24: 10K, PCM_Resistor_SMD_AKL:R_0603_1608Metric, F.Cu at (44.4, 91.2)
- added R25: 10K, PCM_Resistor_SMD_AKL:R_0603_1608Metric, F.Cu at (44.4, 94.0)
- added R26: 10K, PCM_Resistor_SMD_AKL:R_0603_1608Metric, F.Cu at (44.4, 96.7)
- added R27: 10K, PCM_Resistor_SMD_AKL:R_0603_1608Metric, F.Cu at (44.4, 99.4)
- added R28: 10K, PCM_Resistor_SMD_AKL:R_0603_1608Metric, F.Cu at (44.4, 102.1)
- added R29: 10K, PCM_Resistor_SMD_AKL:R_0603_1608Metric, F.Cu at (48.6, 85.8)
- added R3: 10K, PCM_Resistor_SMD_AKL:R_0603_1608Metric, F.Cu at (32.1, 91.2)
- added R30: 10K, PCM_Resistor_SMD_AKL:R_0603_1608Metric, F.Cu at (48.6, 88.5)
- added R31: 10K, PCM_Resistor_SMD_AKL:R_0603_1608Metric, F.Cu at (48.6, 91.2)
- added R32: 10K, PCM_Resistor_SMD_AKL:R_0603_1608Metric, F.Cu at (48.6, 94.0)
- added R33: 10K, PCM_Resistor_SMD_AKL:R_0603_1608Metric, F.Cu at (48.6, 96.7)
- added R34: 10K, PCM_Resistor_SMD_AKL:R_0603_1608Metric, F.Cu at (48.6, 99.4)
- added R35: 10K, PCM_Resistor_SMD_AKL:R_0603_1608Metric, F.Cu at (48.6, 102.1)
- added R36: 10K, PCM_Resistor_SMD_AKL:R_0603_1608Metric, F.Cu at (52.7, 85.8)
- added R37: 10K, PCM_Resistor_SMD_AKL:R_0603_1608Metric, F.Cu at (52.7, 88.5)
- added R38: 10K, PCM_Resistor_SMD_AKL:R_0603_1608Metric, F.Cu at (52.7, 91.2)
- added R39: 10K, PCM_Resistor_SMD_AKL:R_0603_1608Metric, F.Cu at (52.7, 94.0)
- added R4: 680, PCM_Resistor_SMD_AKL:R_0603_1608Metric, F.Cu at (32.1, 94.0)
- added R40: 10K, PCM_Resistor_SMD_AKL:R_0603_1608Metric, F.Cu at (52.7, 96.7)
- added R41: 10K, PCM_Resistor_SMD_AKL:R_0603_1608Metric, F.Cu at (52.7, 99.4)
- added R42: 0R, Resistor_SMD:R_0402_1005Metric, F.Cu at (55.9, 56.7)
- added R43: 14k, Resistor_SMD:R_0402_1005Metric, F.Cu at (55.9, 58.7)
- added R44: 24k, Resistor_SMD:R_0402_1005Metric, F.Cu at (55.9, 60.7)
- added R5: 1.6K, PCM_Resistor_SMD_AKL:R_0603_1608Metric, F.Cu at (32.1, 96.7)
- added R6: 10K, PCM_Resistor_SMD_AKL:R_0603_1608Metric, F.Cu at (32.1, 99.4)
- added R7: 10K, PCM_Resistor_SMD_AKL:R_0603_1608Metric, F.Cu at (32.1, 102.1)
- added R8: 4.7K, PCM_Resistor_SMD_AKL:R_0603_1608Metric, F.Cu at (36.2, 85.8)
- added R9: 4.7K, PCM_Resistor_SMD_AKL:R_0603_1608Metric, F.Cu at (36.2, 88.5)
- added TP1: TestPoint, TestPoint:TestPoint_Pad_D1.0mm, F.Cu at (45.9, 118.3)
- added TP10: TestPoint, TestPoint:TestPoint_Pad_D1.0mm, F.Cu at (55.0, 118.3)
- added TP11: TestPoint, TestPoint:TestPoint_Pad_D1.0mm, F.Cu at (55.0, 121.4)
- added TP12: TestPoint, TestPoint:TestPoint_Pad_D1.0mm, F.Cu at (55.0, 124.5)
- added TP2: TestPoint, TestPoint:TestPoint_Pad_D1.0mm, F.Cu at (45.9, 121.4)
- added TP3: TestPoint, TestPoint:TestPoint_Pad_D1.0mm, F.Cu at (45.9, 124.5)
- added TP4: TestPoint, TestPoint:TestPoint_Pad_D1.0mm, F.Cu at (48.9, 118.3)
- added TP5: TestPoint, TestPoint:TestPoint_Pad_D1.0mm, F.Cu at (48.9, 121.4)
- added TP6: TestPoint, TestPoint:TestPoint_Pad_D1.0mm, F.Cu at (48.9, 124.5)
- added TP7: TestPoint, TestPoint:TestPoint_Pad_D1.0mm, F.Cu at (52.0, 118.3)
- added TP8: TestPoint, TestPoint:TestPoint_Pad_D1.0mm, F.Cu at (52.0, 121.4)
- added TP9: TestPoint, TestPoint:TestPoint_Pad_D1.0mm, F.Cu at (52.0, 124.5)
- added U1: ST1S10PUR, Package_DFN_QFN:DFN-8-1EP_4x4mm_P0.8mm_EP2.5x3.6mm, F.Cu at (51.7, 52.8)
- added Y1: X322524MQB4SI, Crystal:Crystal_SMD_Abracon_ABM8AIG-4Pin_3.2x2.5mm, F.Cu at (47.0, 105.7)
- added Y2: X322524MQB4SI, Crystal:Crystal_SMD_Abracon_ABM8AIG-4Pin_3.2x2.5mm, F.Cu at (47.0, 110.2)
- added Y3: X322524MQB4SI, Crystal:Crystal_SMD_Abracon_ABM8AIG-4Pin_3.2x2.5mm, F.Cu at (47.0, 114.6)
