File: PCIe-USB-hub/PCIe-USB-hub.kicad_pcb (KiCad board)
At the start: 4 copper layers, 166.7 x 111.2 mm, 242 parts, among them J1 USB3_A, J10 USB3_A, J11 USB3_A, J12 Barrel_Jack_MountingPin, J2 USB3_A, J3 USB3_A, J4 USB3_A, J5 PCIexpress_x1, J6 USB3_A, J7 USB3_A, J8 USB3_A, J9 USB3_A, Y1 X322524MQB4SI, Y2 X322524MQB4SI, Y3 X322524MQB4SI

Commit message: натыкал трассировку всех дифф линий, поменял часть местами для удобной трассировки
Parts:
- C7, C8: moved to B.Cu
- moved C67 204.4 mm to (179.1, 51.1), turned to 180 degrees
- moved C65 197.6 mm to (179.1, 52.0), turned to 180 degrees
- moved C89 192.5 mm to (179.8, 67.9), turned to 180 degrees
- moved C97 184.0 mm to (179.8, 67.0), turned to 180 degrees
- moved C88 179.2 mm to (179.4, 84.2), turned to 180 degrees
- moved DD23 173.4 mm to (148.2, 70.3), turned to 45 degrees
- moved C95 173.1 mm to (179.3, 99.3), turned to 180 degrees
- moved C96 171.1 mm to (179.4, 83.3), turned to 180 degrees
- moved TP12 170.7 mm to (139.8, 73.2)
- moved TP11 169.2 mm to (142.0, 73.2)
- moved TP9 168.8 mm to (139.3, 76.9)
- moved C87 167.4 mm to (179.3, 100.3), turned to 180 degrees
- moved TP8 167.3 mm to (138.3, 74.9)
- moved TP7 165.6 mm to (140.3, 75.2)
- moved R77 164.5 mm to (151.5, 72.0), turned to -135 degrees
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Connections:
- net Net-(DD20-U3RXDNU) renamed _USB-host1_TX-
- net Net-(DD20-U3RXDPU) renamed _USB-host1_TX+
- net Net-(DD20-U3TXDN1) renamed _USB-downstream1-TX-
- net Net-(DD20-U3TXDN2) renamed _USB-downstream2-TX-
- net Net-(DD20-U3TXDN3) renamed _USB-downstream3-TX-
- net Net-(DD20-U3TXDN4) renamed _USB-downstream4-TX-
- net Net-(DD20-U3TXDNU) renamed _USB-host1_RX-
- net Net-(DD20-U3TXDP1) renamed _USB-downstream1-TX+
- net Net-(DD20-U3TXDP2) renamed _USB-downstream2-TX+
- net Net-(DD20-U3TXDP3) renamed _USB-downstream3-TX+
- net Net-(DD20-U3TXDP4) renamed _USB-downstream4-TX+
- net Net-(DD20-U3TXDPU) renamed _USB-host1_RX+
- net Net-(DD21-U3RXDNU) renamed _USB-host2_TX-
- net Net-(DD21-U3RXDPU) renamed _USB-host2_TX+
- net Net-(DD21-U3TXDN1) renamed _USB-downstream5-TX-
- net Net-(DD21-U3TXDN2) renamed _USB-downstream6-TX-
- net Net-(DD21-U3TXDN3) renamed _USB-downstream7-TX-
- net Net-(DD21-U3TXDN4) renamed _USB-downstream8-TX-
- net Net-(DD21-U3TXDNU) renamed _USB-host2_RX-
- net Net-(DD21-U3TXDP1) renamed _USB-downstream5-TX+
- net Net-(DD21-U3TXDP2) renamed _USB-downstream6-TX+
- net Net-(DD21-U3TXDP3) renamed _USB-downstream7-TX+
- net Net-(DD21-U3TXDP4) renamed _USB-downstream8-TX+
- net Net-(DD21-U3TXDPU) renamed _USB-host2_RX+
- net Net-(J5-PERn0) renamed _PCIe-TX-
- net Net-(J5-PERp0) renamed _PCIe-TX+
- net Net-(J5-PETn0) renamed _PCIe-RX-
- net Net-(J5-PETp0) renamed _PCIe-RX+
- C64 pad 2: Net-(DD18-U3TXDP3) -> _USB-downstream9-TX+
- C65 pad 2: Net-(DD18-U3RXDP4) -> _USB-downstream10-TX+
- C66 pad 2: Net-(DD18-U3TXDN3) -> _USB-downstream9-TX-
- C67 pad 2: Net-(DD18-U3RXDN4) -> _USB-downstream10-TX-
- DD18 pad 35: USB-host1_TX+ -> USB-host2_TX+
- DD18 pad 36: USB-host1_TX- -> USB-host2_TX-
- DD18 pad 38: USB-host1_RX+ -> USB-host2_RX+
- DD18 pad 39: USB-host1_RX- -> USB-host2_RX-
- DD18 pad 41: USB-host1_D+ -> USB-host2_D+
- DD18 pad 42: USB-host1_D- -> USB-host2_D-
- DD18 pad 44: USB-host2_TX+ -> USB-host1_TX+
- DD18 pad 45: USB-host2_TX- -> USB-host1_TX-
- DD18 pad 47: USB-host2_RX+ -> USB-host1_RX+
- DD18 pad 48: USB-host2_RX- -> USB-host1_RX-
- DD18 pad 50: USB-host2_D+ -> USB-host1_D+
- DD18 pad 51: USB-host2_D- -> USB-host1_D-
- DD18 pad 52: Net-(DD18-U3TXDP3) -> _USB-downstream10-TX+
- DD18 pad 53: Net-(DD18-U3TXDN3) -> _USB-downstream10-TX-
- DD18 pad 55: USB-downstream9-RX+ -> USB-downstream10-RX+
- DD18 pad 56: USB-downstream9-RX- -> USB-downstream10-RX-
- DD18 pad 58: USB-downstream9-D+ -> USB-downstream10-D+
- DD18 pad 59: USB-downstream9-D- -> USB-downstream10-D-
- DD18 pad 61: USB-downstream10-RX+ -> USB-downstream9-RX+
- DD18 pad 62: USB-downstream10-RX- -> USB-downstream9-RX-
- DD18 pad 64: Net-(DD18-U3RXDP4) -> _USB-downstream9-TX+
- DD18 pad 65: Net-(DD18-U3RXDN4) -> _USB-downstream9-TX-
- DD18 pad 67: USB-downstream10-D+ -> USB-downstream9-D+
- DD18 pad 68: USB-downstream10-D- -> USB-downstream9-D-
- DD19 pad 7: +3.3V -> +3.3V_DUAL
- DD22 pad 7: +3.3V -> +3.3V_DUAL
- DD23 pad 7: +3.3V -> +3.3V_DUAL
Routing:
- net USB-downstream10-D-: track 0.00 -> 149.7 mm, vias 0 -> 1
- net USB-downstream10-D+: track 0.00 -> 148.1 mm, vias 0 -> 1
- net USB-downstream10-RX-: track 0.00 -> 129.8 mm, vias 0 -> 2
- net USB-downstream10-RX+: track 0.00 -> 129.0 mm, vias 0 -> 2
- net _USB-downstream10-TX-: track 0.00 -> 117.3 mm, vias 0 -> 2
- net _USB-downstream10-TX+: track 0.00 -> 116.4 mm, vias 0 -> 2
- net USB-downstream9-D-: track 0.00 -> 97.0 mm, vias 0 -> 2
- net USB-downstream9-D+: track 0.00 -> 96.2 mm, vias 0 -> 2
- net USB-downstream9-RX+: track 0.00 -> 84.7 mm, vias 0 -> 2
- net USB-downstream9-RX-: track 0.00 -> 84.6 mm, vias 0 -> 2
- net _USB-downstream9-TX-: track 0.00 -> 81.7 mm, vias 0 -> 2
- net _USB-downstream9-TX+: track 0.00 -> 81.7 mm, vias 0 -> 2
- net USB-downstream5-D-: track 0.00 -> 58.9 mm
- net USB-downstream5-D+: track 0.00 -> 58.2 mm
- net USB-downstream4-D-: track 0.00 -> 56.2 mm
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
Commit message: тык-перетык
Parts:
- added C100: 100nF, Capacitor_SMD:C_0402_1005Metric, F.Cu at (110.2, 93.2)
- added C101: 22uF, Capacitor_SMD:C_0402_1005Metric, F.Cu at (102.8, 105.2)
- added C102: 100nF, Capacitor_SMD:C_0402_1005Metric, F.Cu at (107.4, 116.4)
- added C103: 22uF, Capacitor_SMD:C_0402_1005Metric, B.Cu at (100.6, 100.5)
- added C104: 100nF, Capacitor_SMD:C_0402_1005Metric, B.Cu at (109.0, 96.6)
- added C105: 22uF, Capacitor_SMD:C_0402_1005Metric, B.Cu at (107.7, 102.2)
- added C106: 100nF, Capacitor_SMD:C_0402_1005Metric, B.Cu at (100.6, 97.0)
- added C107: 22uF, Capacitor_SMD:C_0402_1005Metric, B.Cu at (102.4, 94.2)
- added C108: 100nF, Capacitor_SMD:C_0402_1005Metric, B.Cu at (106.1, 94.2)
- added C109: 22uF, Capacitor_SMD:C_0402_1005Metric, B.Cu at (109.0, 97.5)
- added C110: 100nF, Capacitor_SMD:C_0402_1005Metric, B.Cu at (107.2, 94.2)
- added C111: 22uF, Capacitor_SMD:C_0402_1005Metric, B.Cu at (104.8, 94.2)
- added C112: 100nF, Capacitor_SMD:C_0402_1005Metric, B.Cu at (103.6, 94.2)
- added C113: 22uF, Capacitor_SMD:C_0402_1005Metric, B.Cu at (100.8, 95.8)
- added C114: 100nF, Capacitor_SMD:C_0402_1005Metric, B.Cu at (105.3, 102.2)
- added C115: 22uF, Capacitor_SMD:C_0402_1005Metric, B.Cu at (100.6, 98.2)
- added C116: 100nF, Capacitor_SMD:C_0402_1005Metric, B.Cu at (100.7, 99.4)
- added C117: 22uF, Capacitor_SMD:C_0402_1005Metric, B.Cu at (106.2, 102.2)
- added C118: 22uF, Capacitor_SMD:C_0402_1005Metric, B.Cu at (72.9, 96.1)
- added C119: 22uF, Capacitor_SMD:C_0402_1005Metric, B.Cu at (79.3, 96.7)
- added C120: 100nF, Capacitor_SMD:C_0402_1005Metric, B.Cu at (79.5, 90.0)
- added C121: 100nF, Capacitor_SMD:C_0402_1005Metric, B.Cu at (80.5, 90.8)
- added C122: 100nF, Capacitor_SMD:C_0402_1005Metric, B.Cu at (78.7, 89.1)
- added C123: 22uF, Capacitor_SMD:C_0402_1005Metric, B.Cu at (74.7, 88.5)
- added C124: 22uF, Capacitor_SMD:C_0402_1005Metric, B.Cu at (73.0, 90.3)
- added C125: 22uF, Capacitor_SMD:C_0402_1005Metric, B.Cu at (72.2, 91.2)
- added C126: 100nF, Capacitor_SMD:C_0402_1005Metric, B.Cu at (71.3, 94.4)
- added C127: 22uF, Capacitor_SMD:C_0402_1005Metric, B.Cu at (149.5, 83.9)
- added C128: 22uF, Capacitor_SMD:C_0402_1005Metric, B.Cu at (148.7, 83.1)
- added C129: 100nF, Capacitor_SMD:C_0402_1005Metric, B.Cu at (148.8, 76.4)
- added C130: 100nF, Capacitor_SMD:C_0402_1005Metric, B.Cu at (154.3, 76.3)
- added C131: 100nF, Capacitor_SMD:C_0402_1005Metric, B.Cu at (155.2, 77.2)
- added C132: 22uF, Capacitor_SMD:C_0402_1005Metric, B.Cu at (156.8, 78.9)
- added C133: 22uF, Capacitor_SMD:C_0402_1005Metric, B.Cu at (147.9, 82.2)
- added C134: 22uF, Capacitor_SMD:C_0402_1005Metric, B.Cu at (153.5, 84.5)
- added C135: 100nF, Capacitor_SMD:C_0402_1005Metric, B.Cu at (156.1, 82.0)
- added C136: 22uF, Capacitor_SMD:C_0402_1005Metric, B.Cu at (81.2, 91.8)
- added C137: 100nF, Capacitor_SMD:C_0402_1005Metric, F.Cu at (136.0, 64.8)
- added C138: 100nF, Capacitor_SMD:C_0402_1005Metric, B.Cu at (74.6, 97.8)
- added C139: 22uF, Capacitor_SMD:C_0402_1005Metric, B.Cu at (80.2, 95.8)
- added C140: 22uF, Capacitor_SMD:C_0402_1005Metric, B.Cu at (76.8, 87.5)
- added C141: 100nF, Capacitor_SMD:C_0402_1005Metric, B.Cu at (78.0, 88.5)
- added C142: 100nF, Capacitor_SMD:C_0402_1005Metric, B.Cu at (73.8, 89.5)
- added C143: 22uF, Capacitor_SMD:C_0402_1005Metric, B.Cu at (71.3, 92.0)
- added C144: 100nF, Capacitor_SMD:C_0402_1005Metric, B.Cu at (72.1, 95.2)
- added C145: 100nF, Capacitor_SMD:C_0402_1005Metric, F.Cu at (77.8, 111.2)
- added C146: 22uF, Capacitor_SMD:C_0402_1005Metric, B.Cu at (151.4, 85.6)
- added C147: 22uF, Capacitor_SMD:C_0402_1005Metric, B.Cu at (148.3, 77.5)
- added C148: 100nF, Capacitor_SMD:C_0402_1005Metric, B.Cu at (146.9, 81.3)
- added C149: 100nF, Capacitor_SMD:C_0402_1005Metric, B.Cu at (150.2, 84.6)
- added C150: 22uF, Capacitor_SMD:C_0402_1005Metric, B.Cu at (153.4, 75.5)
- added C151: 100nF, Capacitor_SMD:C_0402_1005Metric, B.Cu at (150.6, 75.3)
- added C152: 22uF, Capacitor_SMD:C_0402_1005Metric, B.Cu at (156.9, 81.1)
- added C153: 100nF, Capacitor_SMD:C_0402_1005Metric, B.Cu at (154.4, 83.6)
- added G***: LOGO, LOGO, F.Cu at (159.1, 39.0)
- added G***: LOGO, LOGO, F.Cu at (114.2, 81.5)
- added G***: LOGO, LOGO, F.Cu at (135.6, 39.6)
- added G***: LOGO, LOGO, B.Cu at (90.4, 53.8)
- added G***: LOGO, LOGO, B.Cu at (150.9, 52.5)
- added L10: 0.68uH, Inductor_SMD:L_Cenker_CKCS4020, F.Cu at (138.9, 63.5)
- added L8: 0.68uH, Inductor_SMD:L_Cenker_CKCS4020, F.Cu at (104.6, 114.9)
- added L9: 0.68uH, Inductor_SMD:L_Cenker_CKCS4020, F.Cu at (74.8, 112.6)
- added kibuzzard-67F2EEE1: G***, kibuzzard-67F2EEE1, F.Cu at (84.4, 58.0)
- moved DD1 164.0 mm to (49.4, 47.4), turned to 180 degrees
- moved R4 155.6 mm to (49.8, 44.7), turned to 180 degrees
- moved R81 155.2 mm to (153.2, 67.3), turned to 135 degrees
- moved C13 154.1 mm to (47.6, 47.7), turned to 90 degrees
- moved R2 151.4 mm to (49.8, 45.6), turned to 180 degrees
- moved R83 148.3 mm to (144.0, 69.4), turned to -135 degrees
- moved C33 146.6 mm to (81.8, 49.9), turned to -90 degrees
- moved C27 144.3 mm to (79.1, 50.6), turned to 180 degrees
- moved DD2 142.0 mm to (179.8, 55.0)
- moved C18 141.7 mm to (47.6, 63.1), turned to 90 degrees
- moved C37 141.4 mm to (103.6, 50.5), turned to -90 degrees
- moved DD16 140.1 mm to (100.0, 47.9), turned to 180 degrees
- moved DD3 140.0 mm to (49.4, 62.8), turned to 180 degrees
- moved C31 138.8 mm to (100.9, 51.2), turned to 180 degrees
- moved R64 136.3 mm to (140.8, 69.5), turned to -45 degrees
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Connections:
- C13 pad 1: OCI10B -> +5V_5
- C14 pad 1: OCI10B -> +5V_5
- C18 pad 1: OCI1B -> +5V_1
- C19 pad 1: OCI1B -> +5V_1
- C20 pad 1: OCI3B -> +5V_2
- C21 pad 1: OCI3B -> +5V_2
- C22 pad 1: OCI5B -> +5V_3
- C23 pad 1: OCI5B -> +5V_3
- C24 pad 1: OCI7B -> +5V_4
- C25 pad 1: OCI7B -> +5V_4
- C41 pad 1: OCI1B -> +5V_1
- C42 pad 1: OCI3B -> +5V_2
- C43 pad 1: OCI5B -> +5V_3
- C44 pad 1: OCI7B -> +5V_4
- C45 pad 1: OCI10B -> +5V_5
- C48 pad 1: OCI1B -> +5V_1
- C49 pad 1: OCI3B -> +5V_2
- C50 pad 1: OCI5B -> +5V_3
- C51 pad 1: OCI7B -> +5V_4
- C52 pad 1: OCI10B -> +5V_5
- C55 pad 1: OCI1B -> +5V_1
- C56 pad 1: OCI3B -> +5V_2
- C57 pad 1: OCI5B -> +5V_3
- C58 pad 1: OCI7B -> +5V_4
- C59 pad 1: OCI10B -> +5V_5
- DD1 pad 3: Net-(DD1-#FAULT) -> OCI9B
- DD1 pad 6: OCI10B -> +5V_5
- DD10 pad 3: Net-(DD10-#FAULT) -> OCI8B
- DD10 pad 6: OCI7B -> +5V_4
- DD18 pad 12: unconnected-(DD18-VDD10_2-Pad12) -> 1.05V
- DD18 pad 15: unconnected-(DD18-VDD33_1-Pad15) -> +3.3V_DUAL
- DD18 pad 22: OCI10B -> OCI9B
- DD18 pad 28: unconnected-(DD18-VDD10_3-Pad28) -> 1.05V
- DD18 pad 29: unconnected-(DD18-VDD33_2-Pad29) -> +3.3V_DUAL
- DD18 pad 32: unconnected-(DD18-AVDD33_2-Pad32) -> Net-(DD18-AVDD33_1)
- DD18 pad 37: unconnected-(DD18-VDD10_4-Pad37) -> 1.05V
- DD18 pad 40: unconnected-(DD18-VDD33_3-Pad40) -> +3.3V_DUAL
- DD18 pad 43: unconnected-(DD18-VDD10_5-Pad43) -> 1.05V
- DD18 pad 46: unconnected-(DD18-VDD10_6-Pad46) -> 1.05V
- DD18 pad 49: unconnected-(DD18-VDD33_4-Pad49) -> +3.3V_DUAL
- DD18 pad 54: unconnected-(DD18-VDD10_7-Pad54) -> 1.05V
- DD18 pad 57: unconnected-(DD18-VDD33_5-Pad57) -> +3.3V_DUAL
- DD18 pad 6: unconnected-(DD18-AVDD33_1-Pad6) -> Net-(DD18-AVDD33_1)
- DD18 pad 60: unconnected-(DD18-VDD10_8-Pad60) -> 1.05V
- DD18 pad 63: unconnected-(DD18-VDD10_9-Pad63) -> 1.05V
- DD18 pad 66: unconnected-(DD18-VDD33_6-Pad66) -> +3.3V_DUAL
- DD18 pad 9: unconnected-(DD18-VDD10_1-Pad9) -> 1.05V
- DD2 pad 3: Net-(DD2-#FAULT) -> OCI10B
- DD2 pad 6: OCI10B -> +5V_5
- DD20 pad 11: unconnected-(DD20-VDD10_2-Pad11) -> 1.05V
- DD20 pad 14: unconnected-(DD20-VDD10_3-Pad14) -> 1.05V
- DD20 pad 17: unconnected-(DD20-VDD33_2-Pad17) -> +3.3V_DUAL
- DD20 pad 22: unconnected-(DD20-VDD10_4-Pad22) -> 1.05V
- DD20 pad 25: unconnected-(DD20-VDD33_3-Pad25) -> +3.3V_DUAL
- DD20 pad 28: unconnected-(DD20-VDD10_5-Pad28) -> 1.05V
- DD20 pad 31: unconnected-(DD20-VDD10_6-Pad31) -> 1.05V
- DD20 pad 34: unconnected-(DD20-VDD33_4-Pad34) -> +3.3V_DUAL
- DD20 pad 42: unconnected-(DD20-VDD33_5-Pad42) -> +3.3V_DUAL
- DD20 pad 47: unconnected-(DD20-VDD10_7-Pad47) -> 1.05V
- DD20 pad 5: unconnected-(DD20-VDD10_1-Pad5) -> 1.05V
- DD20 pad 50: unconnected-(DD20-AVDD33R-Pad50) -> Net-(DD20-AVDD33)
- DD20 pad 55: OCI1B -> OCI2B
- DD20 pad 59: OCI3B -> OCI4B
- DD20 pad 61: unconnected-(DD20-VDD33_6-Pad61) -> +3.3V_DUAL
- DD20 pad 64: unconnected-(DD20-VDD10_8-Pad64) -> 1.05V
- DD20 pad 67: unconnected-(DD20-VDD10_9-Pad67) -> 1.05V
- DD20 pad 70: unconnected-(DD20-VDD10_10-Pad70) -> 1.05V
- DD20 pad 71: unconnected-(DD20-AVDD33-Pad71) -> Net-(DD20-AVDD33)
- DD20 pad 76: unconnected-(DD20-VDD33_7-Pad76) -> +3.3V_DUAL
- DD20 pad 8: unconnected-(DD20-VDD33_1-Pad8) -> +3.3V_DUAL
- DD21 pad 11: unconnected-(DD21-VDD10_2-Pad11) -> 1.05V
- DD21 pad 14: unconnected-(DD21-VDD10_3-Pad14) -> 1.05V
- DD21 pad 17: unconnected-(DD21-VDD33_2-Pad17) -> +3.3V_DUAL
- DD21 pad 22: unconnected-(DD21-VDD10_4-Pad22) -> 1.05V
- DD21 pad 25: unconnected-(DD21-VDD33_3-Pad25) -> +3.3V_DUAL
- DD21 pad 28: unconnected-(DD21-VDD10_5-Pad28) -> 1.05V
- DD21 pad 31: unconnected-(DD21-VDD10_6-Pad31) -> 1.05V
- DD21 pad 34: unconnected-(DD21-VDD33_4-Pad34) -> +3.3V_DUAL
- DD21 pad 42: unconnected-(DD21-VDD33_5-Pad42) -> +3.3V_DUAL
- DD21 pad 47: unconnected-(DD21-VDD10_7-Pad47) -> 1.05V
- DD21 pad 5: unconnected-(DD21-VDD10_1-Pad5) -> 1.05V
- DD21 pad 50: unconnected-(DD21-AVDD33R-Pad50) -> Net-(DD21-AVDD33)
- DD21 pad 55: OCI5B -> OCI6B
- DD21 pad 59: OCI7B -> OCI8B
- DD21 pad 61: unconnected-(DD21-VDD33_6-Pad61) -> +3.3V_DUAL
- DD21 pad 64: unconnected-(DD21-VDD10_8-Pad64) -> 1.05V
- DD21 pad 67: unconnected-(DD21-VDD10_9-Pad67) -> 1.05V
- DD21 pad 70: unconnected-(DD21-VDD10_10-Pad70) -> 1.05V
- DD21 pad 71: unconnected-(DD21-AVDD33-Pad71) -> Net-(DD21-AVDD33)
- DD21 pad 76: unconnected-(DD21-VDD33_7-Pad76) -> +3.3V_DUAL
- DD21 pad 8: unconnected-(DD21-VDD33_1-Pad8) -> +3.3V_DUAL
- DD3 pad 3: Net-(DD3-#FAULT) -> OCI1B
- DD3 pad 6: OCI1B -> +5V_1
- DD4 pad 3: Net-(DD4-#FAULT) -> OCI2B
- DD4 pad 6: OCI1B -> +5V_1
- DD5 pad 3: Net-(DD5-#FAULT) -> OCI3B
- DD5 pad 6: OCI3B -> +5V_2
- DD6 pad 3: Net-(DD6-#FAULT) -> OCI4B
- DD6 pad 6: OCI3B -> +5V_2
- DD7 pad 3: Net-(DD7-#FAULT) -> OCI5B
- DD7 pad 6: OCI5B -> +5V_3
- DD8 pad 3: Net-(DD8-#FAULT) -> OCI6B
- DD8 pad 6: OCI5B -> +5V_3
- DD9 pad 3: Net-(DD9-#FAULT) -> OCI7B
- DD9 pad 6: OCI7B -> +5V_4
- L2 pad 2: OCI1B -> +5V_1
- L3 pad 2: OCI3B -> +5V_2
- L4 pad 2: OCI5B -> +5V_3
- L5 pad 2: OCI7B -> +5V_4
- L6 pad 2: OCI10B -> +5V_5
- R10 pad 1: Net-(DD7-#FAULT) -> OCI5B
- R10 pad 2: OCI5B -> +5V_3
- R11 pad 1: Net-(DD8-#FAULT) -> OCI6B
- R11 pad 2: OCI5B -> +5V_3
- R12 pad 1: Net-(DD9-#FAULT) -> OCI7B
- R12 pad 2: OCI7B -> +5V_4
- R13 pad 1: Net-(DD10-#FAULT) -> OCI8B
- R13 pad 2: OCI7B -> +5V_4
- R2 pad 1: Net-(DD1-#FAULT) -> OCI9B
- R2 pad 2: OCI10B -> +5V_5
- R3 pad 1: Net-(DD2-#FAULT) -> OCI10B
- R3 pad 2: OCI10B -> +5V_5
- R33 pad 2: OCI1B -> +5V_1
- R35 pad 2: OCI3B -> +5V_2
- R37 pad 2: OCI5B -> +5V_3
- R39 pad 2: OCI7B -> +5V_4
- R41 pad 2: OCI10B -> +5V_5
- R46 pad 1: OCI10B -> OCI9B
- R57 pad 2: OCI1B -> OCI2B
- R59 pad 2: OCI3B -> OCI4B
- R6 pad 1: Net-(DD3-#FAULT) -> OCI1B
- R6 pad 2: OCI1B -> +5V_1
- R65 pad 2: OCI5B -> OCI6B
- R67 pad 2: OCI7B -> OCI8B
- R7 pad 1: Net-(DD4-#FAULT) -> OCI2B
- R7 pad 2: OCI1B -> +5V_1
- R8 pad 1: Net-(DD5-#FAULT) -> OCI3B
- R8 pad 2: OCI3B -> +5V_2
- R9 pad 1: Net-(DD6-#FAULT) -> OCI4B
- R9 pad 2: OCI3B -> +5V_2
Routing:
- net 1.05V: track 0.00 -> 339.1 mm, vias 0 -> 32
- net +12V: track 0.00 -> 160.4 mm, vias 0 -> 45
- net +5V_5: track 0.00 -> 156.0 mm, vias 0 -> 18
- net Earth: track 0.00 -> 154.7 mm, vias 0 -> 442
- net +3.3V_DUAL: track 0.00 -> 142.1 mm, vias 0 -> 99
- net OCI9B: track 0.00 -> 137.2 mm, vias 0 -> 3
- net PPON9: track 0.00 -> 137.1 mm, vias 0 -> 4
- net OCI10B: track 0.00 -> 134.0 mm, vias 0 -> 2
- net OCI1B: track 0.00 -> 133.2 mm, vias 0 -> 3
- net OCI5B: track 0.00 -> 127.3 mm, vias 0 -> 2
- net PPON1: track 0.00 -> 126.7 mm, vias 0 -> 3
- net PPON10: track 0.00 -> 117.1 mm, vias 0 -> 2
- net PPON6: track 0.00 -> 110.4 mm, vias 0 -> 2
- net OCI6B: track 0.00 -> 104.9 mm, vias 0 -> 2
- net PPON5: track 0.00 -> 101.6 mm, vias 0 -> 2
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- added copper zone on B.Cu, net +12V
- added copper zone on F.Cu, net +12V
- added copper zone on In2.Cu, net +12V
- added copper zone on B.Cu, net +3.3V
- added copper zone on F.Cu, net +3.3V
- added copper zone on B.Cu, net +3.3V_DUAL
- added copper zone on F.Cu, net +3.3V_DUAL
- added copper zone on In2.Cu, net +3.3V_DUAL
- added copper zone on F.Cu, net +5V_1
- added copper zone on In2.Cu, net +5V_1
- added copper zone on F.Cu, net +5V_2
- added copper zone on In2.Cu, net +5V_2
- added copper zone on F.Cu, net +5V_3
- added copper zone on In2.Cu, net +5V_3
- added copper zone on F.Cu, net +5V_4
- added copper zone on In2.Cu, net +5V_4
- added copper zone on F.Cu, net +5V_5
- added copper zone on In2.Cu, net +5V_5
- added copper zone on In2.Cu, net 1.05V
- added copper zone on B.Cu, net Earth
- added copper zone on F.Cu, net Earth
- added copper zone on In1.Cu, net Earth
- added copper zone on F.Cu, net Net-(DD12-SW)
Other:
- board text added: "by @madjogger"
- board text added: "🍪 Раздельное питание на каждый порт"
- board text added: "🍪 Чипы UPD720210 и UPD720201"
