File: PCIe-USB-hub/PCIe-USB-hub.kicad_sch (KiCad schematic)
At the start: 22 parts, among them J1 PCIexpress_x1, J2 USB3_A_Stacked, J3 USB3_A_Stacked, J4 USB3_A_Stacked, J5 USB3_A_Stacked, J6 USB3_A_Stacked, J7 Barrel_Jack_MountingPin

Commit message: Чут чут модифицировал
Parts:
- added C55, C56, C58, C61, C63, C66, C68: 22uF, Capacitor_SMD:C_0402_1005Metric, symbol Device:C
- added C57, C62, C67: 100nF, Capacitor_SMD:C_0402_1005Metric, symbol Device:C
- added C59, C60, C64, C65: 22uF, Capacitor_SMD:C_0805_2012Metric, symbol Device:C
- added DD10, DD9: ST1S10PUR, Package_DFN_QFN:DFN-8-1EP_4x4mm_P0.8mm_EP2.5x3.6mm, symbol Regulator_Switching:ST1S10PUR
- added DD7: ~, SY8843QWC:SY8843QWC, symbol SY8843QWC:SY8843QWC
- added L2: 0.68uH, Inductor_SMD:L_Cenker_CKCS4020, symbol Device:L
- added L3, L4: 3.3uH VLS5045EX-3R3N, PCM_4ms_Inductor:COIL_5040, symbol Device:L
- added R42, R45, R46, R49: 0R, Resistor_SMD:R_0402_1005Metric, symbol Device:R
- added R43: 51.1k, Resistor_SMD:R_0402_1005Metric, symbol Device:R
- added R44: 68k, Resistor_SMD:R_0402_1005Metric, symbol Device:R
- added R47, R50: 4.7k, Resistor_SMD:R_0402_1005Metric, symbol Device:R
- added R48, R51: 1.5k, Resistor_SMD:R_0402_1005Metric, symbol Device:R
Connections:
- net Earth: now also J1.A12 (GND), J1.A15 (GND), J1.A18 (GND), J1.A4 (GND), J1.B13 (GND), J1.B16 (GND), J1.B18 (GND), J1.B4 (GND), J1.B7 (GND), C55.2, C56.2, C57.2, C58.2, C59.2, C60.2, C61.2, C62.2, C63.2, C64.2, C65.2, C66.2, C67.2, C68.2, DD10.4 (AGND), DD10.5 (SYNC), DD10.8 (PGND), DD10.9 (PADGND), DD7.7 (GND), DD9.4 (AGND), DD9.5 (SYNC), DD9.8 (PGND), DD9.9 (PADGND), R44.1, R48.1, R51.1
- net +3.3V: now reaches J1.A10 (+3.3V)
- net +3.3V: now also J1.A9 (+3.3V), J1.B8 (+3.3V), C55.1, DD7.5 (IN), R42.1
- net +12V: now reaches J1.A2 (+12V)
- net +12V: now also J1.A3 (+12V), J1.B1 (+12V), J1.B2 (+12V), J1.B3 (+12V), C59.1, C60.1, C64.1, C65.1, DD10.1 (VINA), DD10.6 (VINSW), DD9.1 (VINA), DD9.6 (VINSW), R45.1, R49.1
- net at J1.B10 (+3.3V_aux): now also R46.1
- new net: DD9.2 (INH), R45.2
- new net: DD9.3 (FB), R47.1, R48.2
- new net: DD9.7 (SW), L3.1
- new net: DD7.1 (FB), R43.1, R44.2
- new net: DD7.4 (EN), R42.2
- new net: DD7.6 (LX), L2.1
- new net: DD10.2 (INH), R49.2
- new net: DD10.3 (FB), R50.1, R51.2
- new net: DD10.7 (SW), L4.1
- new net +3.3V aux: R46.2
- new net +3.3V_DUAL: C61.1, C62.1, C63.1, C66.1, C67.1, C68.1, L3.2, L4.2, R47.2, R50.2
- new net 1.05V: C56.1, C57.1, C58.1, DD7.2 (OUT), L2.2, R43.2
Other:
- note added: "1.05V"
- note added: "1.05В 3А"
- note added: "3.3V"
- note added: "3.3В 3А"
- moved on the sheet: J7

Commit message: Доделал схему, сделал контур платы и расстановку предварительную USB портов
Parts:
- added C69, C70, C74, C75, C79, C80, C84, C85: 22uF, Capacitor_SMD:C_0805_2012Metric, symbol Device:C
- added C71, C73, C76, C78, C81, C83, C86, C88: 22uF, Capacitor_SMD:C_0402_1005Metric, symbol Device:C
- added C72, C77, C82, C87, C90, C91, C92, C93, C94, C95, C96, C97, C98, C99: 100nF, Capacitor_SMD:C_0402_1005Metric, symbol Device:C
- added C89: EEEFK1E151P, Capacitor_SMD:C_Elec_8x10.2, symbol Device:C_Polarized
- added DD11, DD12, DD13, DD14: ST1S10PUR, Package_DFN_QFN:DFN-8-1EP_4x4mm_P0.8mm_EP2.5x3.6mm, symbol Regulator_Switching:ST1S10PUR
- added DD15, DD16, DD17, DD18, DD19, DD20, DD21, DD22, DD23: TPS2552DRVR, Package_SON:WSON-6-1EP_2x2mm_P0.65mm_EP1x1.6mm, symbol TPS2552DRVR:TPS2552DRVR
- added L5, L6, L7, L8: 3.3uH VLS5045EX-3R3N, PCM_4ms_Inductor:COIL_5040, symbol Device:L
- added R52, R55, R58, R61: 0R, Resistor_SMD:R_0402_1005Metric, symbol Device:R
- added R53, R56, R59, R62: 43k, Resistor_SMD:R_0402_1005Metric, symbol Device:R
- added R54, R57, R60, R63: 8.2k, Resistor_SMD:R_0402_1005Metric, symbol Device:R
- added R64, R66, R68, R69, R72, R73, R76, R77, R80, R81: 100k, Resistor_SMD:R_0402_1005Metric, symbol Device:R
- added R65, R67, R70, R71, R74, R75, R78, R79, R82, R83: 20k, Resistor_SMD:R_0402_1005Metric, symbol Device:R
- R50: value 4.7k -> 43k
- R51: value 1.5k -> 8.2k
Connections:
- net +12V: now also J7.1, C69.1, C70.1, C74.1, C75.1, C79.1, C80.1, C84.1, C85.1, C89.1, DD11.1 (VINA), DD11.6 (VINSW), DD12.1 (VINA), DD12.6 (VINSW), DD13.1 (VINA), DD13.6 (VINSW), DD14.1 (VINA), DD14.6 (VINSW), R52.1, R55.1, R58.1, R61.1
- net +3.3V_DUAL: no longer C66.1, C67.1, C68.1, L4.2, R50.2
- net +5V_USB1: now also DD3.1 (OUT)
- net +5V_USB10: now also DD23.1 (OUT)
- net +5V_USB2: now also DD15.1 (OUT)
- net +5V_USB3: now also DD16.1 (OUT)
- net +5V_USB4: now also DD17.1 (OUT)
- net +5V_USB5: now also DD18.1 (OUT)
- net +5V_USB6: now also DD19.1 (OUT)
- net +5V_USB7: now also DD20.1 (OUT)
- net +5V_USB8: now also DD21.1 (OUT)
- net +5V_USB9: now also DD22.1 (OUT)
- net Earth: now also DD3.5 (GND), DD3.7 (EP), J7.2, C69.2, C70.2, C71.2, C72.2, C73.2, C74.2, C75.2, C76.2, C77.2, C78.2, C79.2, C80.2, C81.2, C82.2, C83.2, C84.2, C85.2, C86.2, C87.2, C88.2, C89.2, C90.2, C91.2, C92.2, C93.2, C94.2, C95.2, C96.2, C97.2, C98.2, C99.2, DD11.4 (AGND), DD11.5 (SYNC), DD11.8 (PGND), DD11.9 (PADGND), DD12.4 (AGND), DD12.5 (SYNC), DD12.8 (PGND), DD12.9 (PADGND), DD13.4 (AGND), DD13.5 (SYNC), DD13.8 (PGND), DD13.9 (PADGND), DD14.4 (AGND), DD14.5 (SYNC), DD14.8 (PGND), DD14.9 (PADGND), DD15.5 (GND), DD15.7 (EP), DD16.5 (GND), DD16.7 (EP), DD17.5 (GND), DD17.7 (EP), DD18.5 (GND), DD18.7 (EP), DD19.5 (GND), DD19.7 (EP), DD20.5 (GND), DD20.7 (EP), DD21.5 (GND), DD21.7 (EP), DD22.5 (GND), DD22.7 (EP), DD23.5 (GND), DD23.7 (EP), R54.1, R57.1, R60.1, R63.1, R65.2, R67.2, R70.2, R71.2, R74.2, R75.2, R78.2, R79.2, R82.2, R83.2
- net at DD3.2 (ILIM): now also R65.1
- net at DD3.3 (#FAULT): now also R64.1
- net PPON1: now reaches DD3.6 (EN)
- new net: DD23.3 (#FAULT), R81.1
- new net: DD20.2 (ILIM), R78.1
- new net: DD15.2 (ILIM), R67.1
- new net: DD21.2 (ILIM), R79.1
- new net: DD21.3 (#FAULT), R77.1
- new net: DD14.3 (FB), R62.1, R63.2
- new net: DD18.3 (#FAULT), R72.1
- new net: DD22.2 (ILIM), R82.1
- new net: DD22.3 (#FAULT), R80.1
- new net: DD12.3 (FB), R56.1, R57.2
- new net: DD14.7 (SW), L8.1
- new net: DD20.3 (#FAULT), R76.1
- new net: DD18.2 (ILIM), R74.1
- new net: DD13.3 (FB), R59.1, R60.2
- new net: DD16.2 (ILIM), R70.1
- new net: DD11.7 (SW), L5.1
- new net: DD16.3 (#FAULT), R68.1
- new net: DD17.2 (ILIM), R71.1
- new net: DD11.3 (FB), R53.1, R54.2
- new net: DD23.2 (ILIM), R83.1
- new net: DD12.7 (SW), L6.1
- new net: DD13.7 (SW), L7.1
- new net: DD11.2 (INH), R52.2
- new net: DD13.2 (INH), R58.2
- new net: DD17.3 (#FAULT), R69.1
- new net: DD19.2 (ILIM), R75.1
- new net: DD19.3 (#FAULT), R73.1
- new net: DD12.2 (INH), R55.2
- new net: DD14.2 (INH), R61.2
- new net: DD15.3 (#FAULT), R66.1
- new net +5V_1: C66.1, C67.1, C68.1, C90.1, C91.1, DD15.6 (EN), DD3.6 (EN), L4.2, R50.2, R64.2, R66.2
- new net +5V_2: C71.1, C72.1, C73.1, C92.1, C93.1, DD16.6 (EN), DD17.6 (EN), L5.2, R53.2, R68.2, R69.2
- new net +5V_3: C76.1, C77.1, C78.1, C94.1, C95.1, DD18.6 (EN), DD19.6 (EN), L6.2, R56.2, R72.2, R73.2
- new net +5V_4: C81.1, C82.1, C83.1, C96.1, C97.1, DD20.6 (EN), DD21.6 (EN), L7.2, R59.2, R76.2, R77.2
- new net +5V_5: C86.1, C87.1, C88.1, C98.1, C99.1, DD22.6 (EN), DD23.6 (EN), L8.2, R62.2, R80.2, R81.2
- new net PPON10: DD23.6 (EN)
- new net PPON2: DD15.6 (EN)
- new net PPON3: DD16.6 (EN)
- new net PPON4: DD17.6 (EN)
- new net PPON5: DD18.6 (EN)
- new net PPON6: DD19.6 (EN)
- new net PPON7: DD20.6 (EN)
- new net PPON8: DD21.6 (EN)
- new net PPON9: DD22.6 (EN)
- no-connect marks 5 -> 6
Other:
- removed sheet USB host to USB hub
- note added: "5V_1"
- note added: "5V_2"
- note added: "5V_3"
- note added: "5V_4"
- note added: "5V_5"
- note added: "5В 3А"
- note added: "DC Jack"
- note added: "PCIe"
- note added: "USB UPD720201"
- note added: "USB UPD720210"
- note added: "USB-PWR"
- note added: "control"
- moved on the sheet: C1, C10, C2, C3, C4, C5, C55, C56, C57, C58, C59, C6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
